File: F411 Clock.kicad_sch (KiCad schematic)
At the start: 24 parts, among them J1 USB_C_Receptacle_USB2.0_16P, Q1 DMG3415U, Q2 BC547, SW1 SW_Push, SW2 SW_Push, SW3 SW_Push, SW4 SW_Push, U1 STM32F411CCUx

Commit message: SCH Save: 2 files changed F411 Clock.kicad_pro 0/0/1 F411 Clock.kicad_sch 900/0/46
Parts:
- added BT1: Battery, Battery:BatteryHolder_Keystone_1042_1x18650, symbol Device:Battery
- added BT2: Battery_Cell, Battery:BatteryHolder_Keystone_3034_1x20mm, symbol Device:Battery_Cell
Connections:
- net +BATT: now also BT1.1 (+)
- net GND: now also BT1.2 (-)

Commit message: SCH Save: 2 files changed F411 Clock.kicad_pro 0/0/1 F411 Clock.kicad_sch 176/0/12
Connections:
- net +BATT_2: now also BT2.1 (+)
- net GND: now also BT2.2 (-)
Other:
- moved on the sheet: BT2
Changed lines of the file:
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@@
 	(wire
 		(pts
+			(xy 38.1 115.57) (xy 38.1 121.92)
+		)
+		(stroke
+			(width 0)
+			(type default)
+		)
+	)
+	(wire
+		(pts
 			(xy 43.18 54.61) (xy 45.72 54.61)
 		)
@@
 	(wire
 		(pts
+			(xy 38.1 129.54) (xy 38.1 135.89)
+		)
+		(stroke
+			(width 0)
+			(type default)
+		)
+	)
+	(wire
+		(pts
 			(xy 101.6 180.34) (xy 101.6 184.15)
 		)
@@
 	(symbol
 		(lib_id "Device:Battery_Cell")
-		(at 43.18 137.16 0)
+		(at 38.1 127 0)
 		(unit 1)
 		(body_style 1)
@@
 		(fields_autoplaced yes)
 		(property "Reference" "BT2"
-			(at 46.99 134.0484 0)
+			(at 41.91 123.8884 0)
 			(show_name no)
 			(do_not_autoplace no)
@@
 		)
 		(property "Value" "Battery_Cell"
-			(at 46.99 136.5884 0)
+			(at 41.91 126.4284 0)
 			(show_name no)
 			(do_not_autoplace no)
@@
 		)
 		(property "Footprint" "Battery:BatteryHolder_Keystone_3034_1x20mm"
-			(at 43.18 135.636 90)
+			(at 38.1 125.476 90)
 			(hide yes)
 			(show_name no)
@@
 		)
 		(property "Datasheet" ""
-			(at 43.18 135.636 90)
+			(at 38.1 125.476 90)
 			(hide yes)
 			(show_name no)
@@
 		)
 		(property "Description" "Single-cell battery"
-			(at 43.18 137.16 0)
+			(at 38.1 127 0)
 			(hide yes)
 			(show_name no)
@@
 		)
 		(property "Sim.Device" "V"
-			(at 43.18 137.16 0)
+			(at 38.1 127 0)
 			(hide yes)
 			(show_name no)
@@
 		)
 		(property "Sim.Type" "DC"
-			(at 43.18 137.16 0)
+			(at 38.1 127 0)
 			(hide yes)
 			(show_name no)
@@
 		)
 		(property "Sim.Pins" "1=+ 2=-"
-			(at 43.18 137.16 0)
+			(at 38.1 127 0)
 			(hide yes)
 			(show_name no)
@@
 	)
 	(symbol
+		(lib_id "power:VDD")
+		(at 38.1 115.57 0)
+		(unit 1)
+		(body_style 1)
+		(exclude_from_sim no)
+		(in_bom yes)
+		(on_board yes)
+		(in_pos_files yes)
+		(dnp no)
+		(fields_autoplaced yes)
+		(property "Reference" "#PWR029"
+			(at 38.1 119.38 0)
+			(hide yes)
+			(show_name no)
+			(do_not_autoplace no)
+			(effects
+				(font
+					(size 1.27 1.27)
+				)
+			)
+		)
+		(property "Value" "+BATT_2"
+			(at 38.1 110.49 0)
+			(show_name no)
+			(do_not_autoplace no)
+			(effects
+				(font
+					(size 1.27 1.27)
+				)
+			)
+		)
+		(property "Footprint" ""
+			(at 38.1 115.57 0)
+			(hide yes)
+			(show_name no)
+			(do_not_autoplace no)
+			(effects
+				(font
+					(size 1.27 1.27)
+				)
+			)
+		)
+		(property "Datasheet" ""
+			(at 38.1 115.57 0)
+			(hide yes)
+			(show_name no)
+			(do_not_autoplace no)
+			(effects
+				(font
+					(size 1.27 1.27)
+				)
+			)
+		)
+		(property "Description" "Power symbol creates a global label with name \"VDD\""
+			(at 38.1 115.57 0)
+			(hide yes)
+			(show_name no)
+			(do_not_autoplace no)
+			(effects
+				(font
+					(size 1.27 1.27)
+				)
+			)
+		)
+		(pin "1"
+		)
+		(instances
+			(project "F411 Clock"
+				(path "/6121eee1-efe8-450c-8a4d-3ee76e069735"
+					(reference "#PWR029")
+					(unit 1)
+				)
+			)
+		)
+	)
+	(symbol
 		(lib_id "Device:C_Small")
 		(at 81.28 41.91 0)
@@
 	)
 	(symbol
+		(lib_id "power:GND")
+		(at 38.1 135.89 0)
+		(unit 1)
+		(body_style 1)
+		(exclude_from_sim no)
+		(in_bom yes)
+		(on_board yes)
+		(in_pos_files yes)
+		(dnp no)
+		(fields_autoplaced yes)
+		(property "Reference" "#PWR030"
+			(at 38.1 142.24 0)
+			(hide yes)
+			(show_name no)
+			(do_not_autoplace no)
+			(effects
+				(font
+					(size 1.27 1.27)
+				)
+			)
+		)
+		(property "Value" "GND"
+			(at 38.1 140.97 0)
+			(show_name no)
+			(do_not_autoplace no)
+			(effects
+				(font
+					(size 1.27 1.27)
+				)
+			)
+		)
+		(property "Footprint" ""
+			(at 38.1 135.89 0)
+			(hide yes)
+			(show_name no)
+			(do_not_autoplace no)
+			(effects
+				(font
+					(size 1.27 1.27)
+				)
+			)
+		)
+		(property "Datasheet" ""
+			(at 38.1 135.89 0)
+			(hide yes)
+			(show_name no)
+			(do_not_autoplace no)
+			(effects
+				(font
+					(size 1.27 1.27)
+				)
+			)
+		)
+		(property "Description" "Power symbol creates a global label with name \"GND\" , ground"
+			(at 38.1 135.89 0)
+			(hide yes)
+			(show_name no)
+			(do_not_autoplace no)
+			(effects
+				(font
+					(size 1.27 1.27)
+				)
+			)
+		)
+		(pin "1"
+		)
+		(instances
+			(project "F411 Clock"
+				(path "/6121eee1-efe8-450c-8a4d-3ee76e069735"
+					(reference "#PWR030")
+					(unit 1)
+				)
+			)
+		)
+	)
+	(symbol
 		(lib_id "Display_Character:WC1602A")
 		(at 234.95 77.47 0)
@@
 		(lib_id "Device:Battery")
 		(at 29.21 125.73 0)
+		(mirror y)
 		(unit 1)
 		(body_style 1)
@@
 		(in_pos_files yes)
 		(dnp no)
-		(fields_autoplaced yes)
 		(property "Reference" "BT1"
-			(at 33.02 123.8884 0)
+			(at 25.4 123.8884 0)
 			(show_name no)
 			(do_not_autoplace no)
@@
 		)
 		(property "Value" "Battery"
-			(at 33.02 126.4284 0)
+			(at 25.4 126.4284 0)
 			(show_name no)
 			(do_not_autoplace no)
