File: F411-TableClock.kicad_pcb (KiCad board)
At the start: 2 copper layers, 80.7 x 76 mm, 43 parts, among them J1 USB_C_Receptacle_USB2.0_16P, J2 Conn_01x16_Socket, J4 Conn_01x04_Pin, J5 Conn_01x08_Socket, J6 Conn_01x08_Pin, Q1 DMG3415U, Q2 BC547, SW1 SW_Push, SW2 SW_Push, SW3 SW_Push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

Commit message: DHT added F411 table clock
Parts:
- removed J6: Conn_01x08_Pin, Connector_PinHeader_2.54mm:PinHeader_1x08_P2.54mm_Vertical
- added J4: Conn_01x09_Socket, Connector_PinSocket_2.54mm:PinSocket_1x09_P2.54mm_Vertical, F.Cu at (115.5, 83.5)
- added R13: 5.2k, Resistor_SMD:R_0805_2012Metric, F.Cu at (150.9, 96.6)
- added U3: AM2302, Sensor:ASAIR_AM2302_P2.54mm_Vertical, F.Cu at (149.7, 92.4)
- J5: value Conn_01x08_Socket -> Conn_01x09_Socket; footprint Connector_PinSocket_2.54mm:PinSocket_1x08_P2.54mm_Vertical -> Connector_PinHeader_2.54mm:PinHeader_1x09_P2.54mm_Vertical; moved to B.Cu
- moved J5 39.5 mm to (115.2, 123.2), turned to -90 degrees
- moved R4 4.59 mm to (106.8, 74.0), turned to 0 degrees
- moved R3 4.10 mm to (102.7, 64.8)
- moved R1 2.00 mm to (106.8, 69.8)
- moved R2 1.90 mm to (106.8, 71.9)
- renumbered J4 to J3
Connections:
- J5 pad 1: /UP -> /UP_1
- J5 pad 2: /DOWN -> /DOWN_2
- J5 pad 3: /ENTER -> /ENTER_3
- J5 pad 4: /BACK -> /BACK_4
- J5 pad 5: +BATT -> +BATT_1
- J5 pad 6: +5V -> +5V_1
- J5 pad 7: /EXT -> Net-(J5-Pin_7)
- J5 pad 8: GND -> GND_1
Routing:
- net Net-(J5-Pin_7): track 0.00 -> 54.7 mm
- net Net-(J5-Pin_9): track 0.00 -> 44.4 mm
- net +5V: track 77.6 -> 89.9 mm
- net GND: track 308.1 -> 296.2 mm, vias 100 -> 104
- net /SWDIO: track 73.9 -> 64.1 mm, vias 2 -> 1
- net +3.3V: track 159.4 -> 168.4 mm
- net GND_1: track 155.4 -> 150.2 mm
- net Net-(J1-CC2): track 3.94 -> 7.27 mm
- net /SWCLK: track 59.8 -> 56.9 mm, vias 2 -> 1
- net Net-(J1-CC1): track 4.13 -> 6.88 mm
- net VBUS: track 98.4 -> 97.3 mm
- net Net-(J1-D+-PadA6): track 10.4 -> 9.60 mm
- net /DP: track 13.7 -> 12.9 mm
- net /DN: track 13.0 -> 12.3 mm

Commit message: Refactor code structure for improved readability and maintainability
Parts:
- moved BT1 13.1 mm to (94.1, 122.6)
- moved C5 13.1 mm to (108.4, 136.3)
- moved R13 13.1 mm to (150.6, 109.7)
- moved SW1 13.1 mm to (109.6, 106.4)
- moved SW2 13.1 mm to (118.5, 106.4)
- moved SW3 13.1 mm to (127.3, 106.4)
- moved SW4 13.1 mm to (136.1, 106.4)
- moved U3 13.1 mm to (149.4, 105.5)
- moved J5 12.9 mm to (115.0, 136.1)
Other:
- board size 80.7 x 76 mm -> 81 x 89.1 mm
